File: hardware/pcb/wearable_pcb.kicad_sch (KiCad schematic)
At the start: 3 parts

Commit message: docs: finalize systems design, polymorphic telemetry theory, and Prizzm copyright updates
Other:
- company: FrozenLionMax -> Prizzm
Changed lines of the file:
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@@
   (title_block
     (title "S.P.H.E.R.E. Wearable Biosensor Schematic")
-    (company "FrozenLionMax")
+    (company "Prizzm")
     (comment 1 "ESP32 MCU with MAX30102 PPG and MPU6050 IMU")
   )
